Commit message: Fixed the simulation and added a new map and fixed the automatic SLAM

File: p3dx/p3dx_description/urdf/pioneer3dx.xacro (robot description, xacro)
@@ -18,4 +18,5 @@
 <robot name="pioneer3dx"
 	xmlns:xacro="http://ros.org/wiki/xacro">
+	<xacro:property name="camera_link" value="0.05" />
 	<!-- import all gazebo-customization elements, including gazebo colors -->
 	<xacro:include filename="$(find rubbish_robot_project)/p3dx/p3dx_description/urdf/pioneer3dx.gazebo" />
@@ -156,4 +157,32 @@
 		<child link="center_hubcap"/>
 	</joint>
+	<!-- Camera -->
+	<joint name="camera_joint" type="fixed">
+		<axis xyz="0 1 0" />
+		<origin xyz="${camera_link} 0 0.5" rpy="0 0 0"/>
+		<parent link="base_link"/>
+		<child link="camera_link"/>
+	</joint>
+	<!-- Camera -->
+	<link name="camera_link">
+		<collision>
+		<origin xyz="0 0 0" rpy="0 0 0"/>
+		<geometry>
+		<box size="${camera_link} ${camera_link} ${camera_link}"/>
+		</geometry>
+		</collision>
+		<visual>
+		<origin xyz="0 0 0" rpy="0 0 0"/>
+		<geometry>
+		<box size="${camera_link} ${camera_link} ${camera_link}"/>
+		</geometry>
+		<material name="red"/>
+		</visual>
+		<inertial>
+		<mass value="1e-5" />
+		<origin xyz="0 0 0" rpy="0 0 0"/>
+		<inertia ixx="1e-6" ixy="0" ixz="0" iyy="1e-6" iyz="0" izz="1e-6" />
+		</inertial>
+	</link>
 	<!-- End of Legacy for diff drive plugin
 	https://github.com/ros-simulation/gazebo_ros_pkgs/pull/707/files
